File: testproj/testproj.kicad_pcb (KiCad board)
At the start: 2 copper layers, 0 parts

Commit message: crap
Parts:
- added U1: XC6SLX100-CSG484, mylib:Xilinx_CSG324, F.Cu at (87.0, 116.0)
Routing:
- net (no net): track 0.00 -> 21.0 mm, vias 0 -> 15
- net unconnected-(U1-PadB3): track 0.00 -> 1.97 mm
- net unconnected-(U1-PadB4): track 0.00 -> 1.97 mm
- net unconnected-(U1-PadA4): track 0.00 -> 1.10 mm
- net unconnected-(U1-PadA16): track 0.00 -> 1.00 mm
- net unconnected-(U1-PadA15): track 0.00 -> 1.00 mm
- net TCK: track 0.00 -> 1.00 mm
- net unconnected-(U1-PadA18): track 0.00 -> 0.90 mm
- net unconnected-(U1-PadF12): track 0.00 -> 0.57 mm, vias 0 -> 1
- net unconnected-(U1-PadE13): track 0.00 -> 0.57 mm, vias 0 -> 1
- net TMS: track 0.00 -> 0.57 mm, vias 0 -> 1
- net unconnected-(U1-PadG11): track 0.00 -> 0.57 mm, vias 0 -> 1
- net unconnected-(U1-PadC18): track 0.00 -> 0.57 mm, vias 0 -> 1
- net unconnected-(U1-PadC17): track 0.00 -> 0.57 mm, vias 0 -> 1
- net unconnected-(U1-PadB16): track 0.00 -> 0.57 mm, vias 0 -> 1
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Other:
- rule pad_to_mask_clearance: 0 -> 0.1

Commit message: crap
Parts:
- added REF**: Xilinx_CSG324, mylib:Xilinx_CSG324, F.Cu at (106.8, 106.8)
- moved U1 76.8 mm to (54.5, 46.4)
Routing:
- net (no net): track 21.0 -> 35.0 mm
- net unconnected-(U1-PadC7): track 0.00 -> 3.56 mm, vias 0 -> 1
- net unconnected-(U1-PadC5): track 0.00 -> 3.17 mm, vias 0 -> 1
- net unconnected-(U1-PadC6): track 0.00 -> 2.97 mm, vias 0 -> 1
- net unconnected-(U1-PadC9): track 0.00 -> 2.97 mm, vias 0 -> 1
- net unconnected-(U1-PadC14): track 0.00 -> 2.97 mm, vias 0 -> 1
- net unconnected-(U1-PadC13): track 0.00 -> 2.97 mm, vias 0 -> 1
- net unconnected-(U1-PadC10): track 0.00 -> 2.97 mm, vias 0 -> 1
- net unconnected-(U1-PadC11): track 0.00 -> 2.87 mm, vias 0 -> 1
- net unconnected-(U1-PadC8): track 0.00 -> 2.87 mm, vias 0 -> 1
- net unconnected-(U1-PadC12): track 0.00 -> 2.77 mm, vias 0 -> 1
- net unconnected-(U1-PadC16): track 0.57 -> 2.89 mm
- net unconnected-(U1-PadC17): track 0.57 -> 2.87 mm
- net unconnected-(U1-PadB6): track 0.00 -> 2.27 mm
- net unconnected-(U1-PadC18): track 0.57 -> 2.81 mm
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Other:
- copper layers 2 -> 4

Commit message: progress
Parts:
- removed REF**: Xilinx_CSG324, mylib:Xilinx_CSG324
Routing:
- net (no net): track 35.0 -> 0.00 mm, vias 15 -> 0
- net unconnected-(U1-PadC7): track 3.56 -> 0.00 mm, vias 1 -> 0
- net unconnected-(U1-PadC5): track 3.17 -> 0.00 mm, vias 1 -> 0
- net unconnected-(U1-PadC6): track 2.97 -> 0.00 mm, vias 1 -> 0
- net unconnected-(U1-PadC9): track 2.97 -> 0.00 mm, vias 1 -> 0
- net unconnected-(U1-PadC14): track 2.97 -> 0.00 mm, vias 1 -> 0
- net unconnected-(U1-PadC13): track 2.97 -> 0.00 mm, vias 1 -> 0
- net unconnected-(U1-PadC10): track 2.97 -> 0.00 mm, vias 1 -> 0
- net unconnected-(U1-PadC16): track 2.89 -> 0.00 mm, vias 1 -> 0
- net unconnected-(U1-PadC11): track 2.87 -> 0.00 mm, vias 1 -> 0
- net unconnected-(U1-PadC8): track 2.87 -> 0.00 mm, vias 1 -> 0
- net unconnected-(U1-PadC17): track 2.87 -> 0.00 mm, vias 1 -> 0
- net unconnected-(U1-PadC18): track 2.81 -> 0.00 mm, vias 1 -> 0
- net unconnected-(U1-PadC15): track 2.77 -> 0.00 mm, vias 1 -> 0
- net unconnected-(U1-PadC12): track 2.77 -> 0.00 mm, vias 1 -> 0
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Other:
- board text added: "fuckfuck"
